File: USB-DB9_Adapter.kicad_sch (KiCad schematic)
At the start: 31 parts, among them IC2 STM32G0B1KBU6-N, U2 U_SPANNUNGSREGLERSOT23, X1 USB-1X-2S-PLUG-A-SMD, X4 M09H, X7 SWD_MOSER_CONN_5_POLST

Commit message: Add files via upload
Parts:
- removed C1: 4N7, USB-DB9_Adapter:C0603, symbol USB-DB9_Adapter-eagle-import:CC0603
- removed C2, C3, C4, C5: 1µF, USB-DB9_Adapter:C0603, symbol USB-DB9_Adapter-eagle-import:CC0603
- removed D1: RED, USB-DB9_Adapter:0805_D, symbol USB-DB9_Adapter-eagle-import:D_LED0805_D
- removed D2: GREEN, USB-DB9_Adapter:0805_D, symbol USB-DB9_Adapter-eagle-import:D_LED0805_D
- removed D3, D4, D5: BLUE, USB-DB9_Adapter:0805_D, symbol USB-DB9_Adapter-eagle-import:D_LED0805_D
- removed IC2: STM32G0B1KBU6-N, USB-DB9_Adapter:QFN50P500X500X60-33N, symbol USB-DB9_Adapter-eagle-import:STM32G0B1KBU6-N
- removed R1, R14, R15, R19, R29, R41: 82R, USB-DB9_Adapter:0603, symbol USB-DB9_Adapter-eagle-import:R
- removed R11: 1M, USB-DB9_Adapter:0603, symbol USB-DB9_Adapter-eagle-import:R
- removed R43: 200K, USB-DB9_Adapter:0603, symbol USB-DB9_Adapter-eagle-import:R
- removed R44: 40.2K, USB-DB9_Adapter:0603, symbol USB-DB9_Adapter-eagle-import:R
- removed S2: TASER_KSR, USB-DB9_Adapter:KSR_TASTER, symbol USB-DB9_Adapter-eagle-import:TASER_KSR
- removed TP10, TP11, TP3, TP5, TP6: don't show, USB-DB9_Adapter:TESTPUNKT, symbol USB-DB9_Adapter-eagle-import:TESTPUNKTTESTPUNKT
- removed U2: U_SPANNUNGSREGLERSOT23, USB-DB9_Adapter:SOT23, symbol USB-DB9_Adapter-eagle-import:U_SPANNUNGSREGLERSOT23
- removed VD1: USBLC6-2SC6, USB-DB9_Adapter:SOT-23-6L, symbol USB-DB9_Adapter-eagle-import:USBLC6-2SC6
- removed X1: USB-1X-2S-PLUG-A-SMD, USB-DB9_Adapter:USB-PLUG-A-SMD-2S, symbol USB-DB9_Adapter-eagle-import:USB-1X-2S-PLUG-A-SMD
- removed X4: M09H, USB-DB9_Adapter:M09H, symbol USB-DB9_Adapter-eagle-import:M09H
- removed X7: SWD_MOSER_CONN_5_POLST, USB-DB9_Adapter:SWD_MOSER_CONN_5_POL_.5MM, symbol USB-DB9_Adapter-eagle-import:SWD_MOSER_CONN_5_POLST
Other:
- note removed: "1"
- note removed: "1000-3511"
- note removed: "23.05.19"
- note removed: "A.Jon"
- note removed: "S.Beha"
- note removed: "Service Adapter 4.0"
- note removed: "single supply translating OR gate, als Level Shifter 3V3 von clipper ->5V an ADMU"

Commit message: Add files via upload
Parts:
- added C1: 4N7, USB-DB9_Adapter:C0603, symbol USB-DB9_Adapter-eagle-import:CC0603
- added C2, C3, C4, C5: 1µF, USB-DB9_Adapter:C0603, symbol USB-DB9_Adapter-eagle-import:CC0603
- added D1: RED, USB-DB9_Adapter:0805_D, symbol USB-DB9_Adapter-eagle-import:D_LED0805_D
- added D2: GREEN, USB-DB9_Adapter:0805_D, symbol USB-DB9_Adapter-eagle-import:D_LED0805_D
- added D3, D4, D5: BLUE, USB-DB9_Adapter:0805_D, symbol USB-DB9_Adapter-eagle-import:D_LED0805_D
- added IC2: STM32G0B1KBU6-N, USB-DB9_Adapter:QFN50P500X500X60-33N, symbol USB-DB9_Adapter-eagle-import:STM32G0B1KBU6-N
- added R1, R14, R15, R19, R29, R41: 82R, USB-DB9_Adapter:0603, symbol USB-DB9_Adapter-eagle-import:R
- added R11: 1M, USB-DB9_Adapter:0603, symbol USB-DB9_Adapter-eagle-import:R
- added S2: TASER_KSR, USB-DB9_Adapter:KSR_TASTER, symbol USB-DB9_Adapter-eagle-import:TASER_KSR
- added TP1, TP10, TP11, TP12, TP13, TP14, TP15, TP2, TP3, TP4, TP5, TP6, TP7, TP8, TP9: don't show, USB-DB9_Adapter:TESTPUNKT, symbol USB-DB9_Adapter-eagle-import:TESTPUNKTTESTPUNKT
- added U2: U_SPANNUNGSREGLERSOT23, USB-DB9_Adapter:SOT23, symbol USB-DB9_Adapter-eagle-import:U_SPANNUNGSREGLERSOT23
- added VD1: USBLC6-2SC6, USB-DB9_Adapter:SOT-23-6L, symbol USB-DB9_Adapter-eagle-import:USBLC6-2SC6
- added X1: USB-1X-2S-PLUG-A-SMD, USB-DB9_Adapter:USB-PLUG-A-SMD-2S, symbol USB-DB9_Adapter-eagle-import:USB-1X-2S-PLUG-A-SMD
- added X4: M09H, USB-DB9_Adapter:M09H, symbol USB-DB9_Adapter-eagle-import:M09H
- added X7: SWD_MOSER_CONN_5_POLST, USB-DB9_Adapter:SWD_MOSER_CONN_5_POL_.5MM, symbol USB-DB9_Adapter-eagle-import:SWD_MOSER_CONN_5_POLST
Connections:
- new net: IC2.19 (PA9), TP8.TP
- new net: IC2.17 (PB15), TP12.TP
- new net: IC2.22 (PA11_[PA9]), VD1.1 (I/O_1)
- new net: IC2.23 (PA12_[PA10]), VD1.3 (I/O_2)
- new net: VD1.4 (I/O2), X1.3
- new net: VD1.6 (I/O1), X1.2
- new net: IC2.14 (PA7), R19.1
- new net: D3.A, R19.2
- new net: D1.A, R14.2
- new net: IC2.11 (PA4), R29.1
- new net: D4.A, R29.2
- new net: IC2.18 (PA8), TP9.TP
- new net: IC2.21 (PA10), TP13.TP
- new net: IC2.10 (PA3), TP4.TP
- new net: IC2.12 (PA5), R14.1
- new net: IC2.13 (PA6), R15.1
- new net: IC2.15 (PB0), R41.1
- new net: IC2.24 (PA13), X7.SWDIO (>NAME)
- new net: IC2.25 (PA14-BOOT0), R1.1, X7.SWDCLK (>NAME)
- new net: IC2.27 (PD1), TP6.TP
- new net: IC2.28 (PD2), TP5.TP
- new net: IC2.29 (PD3), TP15.TP
- new net: IC2.30 (PB6), TP2.TP
- new net: IC2.31 (PB7), TP1.TP
- new net: IC2.32 (PB8), TP3.TP
- new net: IC2.6 (PF2-NRST), X7.NRST (>NAME)
- new net: IC2.7 (PA0), TP14.TP
- new net: IC2.9 (PA2), TP7.TP
- new net: R1.2, S2.P$1 (1)
- new net: D5.A, R41.2
- new net: C1.1, R11.1, X1.S1, X1.S2
- new net: D2.A, R15.2
- new net 3V3: C2.1, C3.1, IC2.20 (VDDIO2), IC2.4 (VDD/VDDA), S2.P$2 (3), U2.E (OUT), X7.VDD (>NAME)
- new net BUTTON1: IC2.8 (PA1), X4.6
- new net BUTTON2: IC2.16 (PB1), X4.9
- new net BUTTON3: IC2.1 (PB9), X4.5
- new net DOWN: IC2.2 (PC14-OSC32_IN), X4.2
- new net GND: C1.2, C2.2, C3.2, C4.2, C5.2, D1.C, D2.C, D3.C, D4.C, D5.C, IC2.33 (EP), IC2.5 (VSS/VSSA), R11.2, TP11.TP, U2.B (GND), VD1.2 (GND), X1.4, X4.8, X7.GND (>NAME)
- new net LEFT: IC2.26 (PD0), X4.3
- new net RIGHT: IC2.3 (PC15-OSC32_OUT), X4.4
- new net UP: X4.1
- new net VCC: C4.1, C5.1, TP10.TP, U2.C (IN), VD1.5 (VBUS), X1.1, X4.7
Other:
- note added: "1"
- note added: "1000-3511"
- note added: "23.05.19"
- note added: "A.Jon"
- note added: "S.Beha"
- note added: "Service Adapter 4.0"
- note added: "single supply translating OR gate, als Level Shifter 3V3 von clipper ->5V an ADMU"

Commit message: Add files via upload
Connections:
- net UP: now also IC2.32 (PB8), TP3.TP
Changed lines of the file:
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@@
+		)
+	)
+	(label "UP"
+		(at 170.18 129.54 0)
+		(effects
+			(font
+				(size 1.27 1.27)
+			)
+			(justify left bottom)
 		)
 	)
